Commit message: world state done + some of state

File: src/arm3dof/urdf/threeDOF.urdf (robot description, URDF)
Before this commit: robot threeDOF, 14 links, 13 joints
Links:
- removed link table
- removed link wall
- added link bound; collision box size=4 4 2; visual box size=4 4 2
Joints:
- removed joint attach-table
- removed joint attach-wall
- added joint attach-bound: type fixed, parent world, child bound

Commit message: adding sphere obstacle to urdf

File: src/arm3dof/urdf/threeDOF.urdf (robot description, URDF)
Before this commit: robot threeDOF, 13 links, 12 joints
Links:
- added link sphere_link; visual sphere radius=0.3
Joints:
- added joint attach-sphere: type fixed, parent world, child sphere_link

Commit message: 3dof environment

File: src/arm3dof/urdf/threeDOF.urdf (robot description, URDF)
Before this commit: robot threeDOF, 14 links, 13 joints
Links:
- removed link sphere_link
- added link sphere_link1; visual sphere radius=0.6
- added link sphere_link2; visual sphere radius=0.6
- added link sphere_link3; visual sphere radius=0.6
- added link sphere_link4; visual sphere radius=0.6
Joints:
- removed joint attach-sphere
- added joint attach-sphere1: type fixed, parent world, child sphere_link1
- added joint attach-sphere2: type fixed, parent world, child sphere_link2
- added joint attach-sphere3: type fixed, parent world, child sphere_link3
- added joint attach-sphere4: type fixed, parent world, child sphere_link4
